File: PCB/Esquemáticos-Eagle/Phineas.sch (EAGLE design)
At the start: 11 parts

Commit message: Editando o esquemático phineas
Connections:
- removed net N$15: ARDUINO_NANO1.D3, R5.A, R5.E, SG1.2
- new net N$16: R5.E, SG1.2
- new net N$18: ARDUINO_NANO1.D3, R5.S
Changed lines of the file:
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@@
 </segment>
 </net>
-<net name="N$15" class="0">
+<net name="N$16" class="0">
 <segment>
 <pinref part="SG1" gate="G$1" pin="2"/>
-<pinref part="R5" gate="G$1" pin="A"/>
 <pinref part="R5" gate="G$1" pin="E"/>
-<wire x1="167.64" y1="208.28" x2="167.64" y2="172.72" width="0.1524" layer="91"/>
-<wire x1="167.64" y1="172.72" x2="58.42" y2="172.72" width="0.1524" layer="91"/>
+</segment>
+</net>
+<net name="N$18" class="0">
+<segment>
+<pinref part="R5" gate="G$1" pin="S"/>
+<wire x1="172.72" y1="215.9" x2="172.72" y2="172.72" width="0.1524" layer="91"/>
+<wire x1="172.72" y1="172.72" x2="58.42" y2="172.72" width="0.1524" layer="91"/>
 <pinref part="ARDUINO_NANO1" gate="G$1" pin="D3"/>
 <wire x1="58.42" y1="172.72" x2="58.42" y2="165.1" width="0.1524" layer="91"/>
