File: PCB/Phineas-PCB.brd (EAGLE design)
At the start: 130 x 131.9 mm, 11 parts

Commit message: PCB Phineas
Parts:
- moved R4 53.9 mm to (35.9, 98.9)
- moved R3 53.9 mm to (35.6, 112.7)
- moved R1 41.2 mm to (25.6, 116.7)
- moved R2 31.6 mm to (25.6, 100.3)
- moved BUZZER 20.0 mm to (53.5, 104.1)
- moved PULAR 20.0 mm to (41.5, 33.1)
- moved DESCER 20.0 mm to (84.8, 32.7)
- moved R5 14.1 mm to (109.4, 73.5)
- moved DIS1 10.0 mm to (63.5, 72.2)
- moved ARDUINO_NANO1 10.0 mm to (87.1, 104.6)
- moved RESET 10.0 mm to (101.1, 42.4)
Routing:
- net VCC: track 0.00 -> 271.3 mm
- net GND: track 0.00 -> 238.3 mm
- net N$8: track 0.00 -> 148.6 mm
- net N$4: track 0.00 -> 143.3 mm
- net N$18: track 0.00 -> 133.7 mm
- net N$3: track 0.00 -> 100.9 mm
- net N$2: track 0.00 -> 99.4 mm
- net N$7: track 0.00 -> 81.0 mm
- net N$16: track 0.00 -> 73.2 mm
- net N$5: track 0.00 -> 66.1 mm
- net N$6: track 0.00 -> 64.1 mm
- net N$9: track 0.00 -> 63.0 mm
- net N$13: track 0.00 -> 36.9 mm
- net N$12: track 0.00 -> 35.9 mm
- net N$11: track 0.00 -> 35.4 mm
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- added copper zone on layer 16, net GND
Other:
- board size 130 x 131.9 mm -> 130 x 111.9 mm
