File: Esquematicos/Eagle/Erika.sch (EAGLE design)
At the start: 12 parts

Commit message: Correção do esquemático
Parts:
- removed BOTAO_1, BOTAO_2, BOTAO_3: (no value), switch-omron:10-XX
- removed POTENCIOMETRO_2: EVUE2A, pot:EVUE2A
- added DESCER, PULAR, RESET: (no value), switch-omron:10-XX
- added R3: (no value), rcl:R-US_0204/7
Connections:
- new net GND: ARDUINO_NANO1.GND@1, BUZZER.2, DISPLAY_LCD.GND, DISPLAY_LCD.NC@2, DISPLAY_LCD.R/W, R1.2, R2.1, R3.1, R7.1
- new net N$1: ARDUINO_NANO1.D4, DISPLAY_LCD.D4
- new net N$13: ARDUINO_NANO1.D7, DISPLAY_LCD.D7
- new net N$14: ARDUINO_NANO1.D8, DISPLAY_LCD.RS
- new net N$15: ARDUINO_NANO1.D9, DISPLAY_LCD.E
- new net N$16: ARDUINO_NANO1.D3, POTENCIOMETRO.A
- net N$10: now also PULAR.P1; no longer BOTAO_3.P1
- net N$11: now also R3.2; no longer POTENCIOMETRO_2.S
- net N$12: now also ARDUINO_NANO1.D6, DISPLAY_LCD.D6; no longer ARDUINO_NANO1.GND@1, BOTAO_1.P, BOTAO_2.P, BOTAO_3.P, BUZZER.1, DISPLAY_LCD.GND, DISPLAY_LCD.NC@2, DISPLAY_LCD.R/W, POTENCIOMETRO.A, POTENCIOMETRO_2.A, R1.2, R2.1, R7.1
- net N$2: now also DESCER.P1; no longer BOTAO_1.P1
- net N$3: now also ARDUINO_NANO1.D10, PULAR.P; no longer ARDUINO_NANO1.A7, DISPLAY_LCD.E
- net N$4: now also ARDUINO_NANO1.D11, DESCER.P; no longer ARDUINO_NANO1.A1, DISPLAY_LCD.D4
- net N$5: now also ARDUINO_NANO1.D12, RESET.P; no longer ARDUINO_NANO1.A0, DISPLAY_LCD.D5
- net N$6: now also BUZZER.1, POTENCIOMETRO.S; no longer ARDUINO_NANO1.AREF, DISPLAY_LCD.D6
- net N$7: now also ARDUINO_NANO1.D5, DISPLAY_LCD.D5; no longer ARDUINO_NANO1.3V3, DISPLAY_LCD.D7
- net N$8: now also RESET.P1; no longer BOTAO_2.P1
- net N$9: now also DESCER.S1, PULAR.S1, RESET.S1; no longer BOTAO_1.S, BOTAO_1.S1, BOTAO_2.S, BOTAO_2.S1, BOTAO_3.S, BOTAO_3.S1, BUZZER.2, DISPLAY_LCD.RS, POTENCIOMETRO.E, POTENCIOMETRO.S, POTENCIOMETRO_2.E
Other:
- moved on the sheet: ARDUINO_NANO1, BUZZER, DISPLAY_LCD, POTENCIOMETRO, R1, R2, R7

Commit message: Atualizando a PCB
Parts:
- removed R8: (no value), rcl:R-US_0204/7
Connections:
- net N$9 renamed VCC
Changed lines of the file:
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@@
 <?xml version="1.0" encoding="utf-8"?>
 <!DOCTYPE eagle SYSTEM "eagle.dtd">
-<eagle version="9.3.2">
+<eagle version="9.6.2">
 <drawing>
 <settings>
@@
 </variantdefs>
 <classes>
-<class number="0" name="default" width="0" drill="0">
+<class number="0" name="default" width="0.508" drill="0">
+</class>
+<class number="1" name="alimentação" width="1.016" drill="0">
 </class>
 </classes>
@@
 <part name="R2" library="rcl" library_urn="urn:adsk.eagle:library:334" deviceset="R-US_" device="0204/7" package3d_urn="urn:adsk.eagle:package:23498/2"/>
 <part name="R7" library="rcl" library_urn="urn:adsk.eagle:library:334" deviceset="R-US_" device="0204/7" package3d_urn="urn:adsk.eagle:package:23498/2"/>
-<part name="R8" library="rcl" library_urn="urn:adsk.eagle:library:334" deviceset="R-US_" device="0204/7" package3d_urn="urn:adsk.eagle:package:23498/2"/>
 <part name="R3" library="rcl" library_urn="urn:adsk.eagle:library:334" deviceset="R-US_" device="0204/7" package3d_urn="urn:adsk.eagle:package:23498/2"/>
 <part name="GND1" library="supply1" library_urn="urn:adsk.eagle:library:371" deviceset="GND" device=""/>
@@
 <attribute name="VALUE" x="94.742" y="80.01" size="1.778" layer="96" rot="R90"/>
 </instance>
-<instance part="R8" gate="G$1" x="20.32" y="20.32" smashed="yes">
-<attribute name="NAME" x="16.51" y="21.8186" size="1.778" layer="95"/>
-<attribute name="VALUE" x="16.51" y="17.018" size="1.778" layer="96"/>
-</instance>
 <instance part="R3" gate="G$1" x="50.8" y="149.86" smashed="yes" rot="R270">
 <attribute name="NAME" x="52.2986" y="153.67" size="1.778" layer="95" rot="R270"/>
@@
 </segment>
 </net>
-<net name="GND" class="0">
+<net name="GND" class="1">
 <segment>
 <pinref part="R3" gate="G$1" pin="1"/>
@@
 </segment>
 </net>
-<net name="N$9" class="0">
+<net name="VCC" class="1">
 <segment>
 <pinref part="DISPLAY_LCD" gate="G$1" pin="VCC"/>

Commit message: Incluindo Versão 2 da PCB, se Deus quiser agora tá certo #fé
Parts:
- removed POTENCIOMETRO: EVUE2A, pot:EVUE2A
- removed R7: (no value), rcl:R-US_0204/7
- added POT: (no value), pot:3RP/1610N
- added R4: (no value), rcl:R-US_0207/10
- BUZZER: value F/EE21P -> F/QMB; device buzzer:F/EE21P -> buzzer:F/QMB
- DESCER, PULAR, RESET: device switch-omron:10-XX -> switch-omron:40-XX
- R1, R2, R3: device rcl:R-US_0204/7 -> rcl:R-US_0207/10
- renumbered DISPLAY_LCD to DIS1
Connections:
- net GND: now also BUZZER.-, R1.1, R4.2; no longer BUZZER.2, R1.2, R7.1
- net N$10: now also R3.2; no longer R7.2
- net N$11: now also R4.1; no longer R3.2
- net N$16: now also POT.A; no longer POTENCIOMETRO.A
- net N$2: now also R1.2; no longer R1.1
- net N$6: now also BUZZER.+, POT.S; no longer BUZZER.1, POTENCIOMETRO.S
Other:
- moved on the sheet: R1, R3
