File: Esquematicos/Eagle/Patrick.sch (EAGLE design)
At the start: 11 parts, among them X1 HD44780LCD-1602

Commit message: Atualizacao do esquematico e da PCB
Connections:
- removed net N$14: REG_BRIGHT.2
- net VCC: now also REG_BRIGHT.2
Changed lines of the file:
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@@
 </variantdefs>
 <classes>
-<class number="0" name="default" width="0" drill="0">
+<class number="0" name="default" width="0.508" drill="0">
+</class>
+<class number="1" name="Alimentacao" width="1.016" drill="0">
 </class>
 </classes>
@@
 </busses>
 <nets>
-<net name="VCC" class="0">
+<net name="VCC" class="1">
 <segment>
 <pinref part="P+3" gate="VCC" pin="VCC"/>
 <pinref part="X1" gate="G$1" pin="VDD"/>
-<wire x1="33.02" y1="160.02" x2="33.02" y2="182.88" width="0.1524" layer="91"/>
+<wire x1="33.02" y1="160.02" x2="33.02" y2="177.8" width="0.1524" layer="91"/>
 <pinref part="X1" gate="G$1" pin="A"/>
+<wire x1="33.02" y1="177.8" x2="33.02" y2="182.88" width="0.1524" layer="91"/>
 <wire x1="33.02" y1="182.88" x2="33.02" y2="185.42" width="0.1524" layer="91"/>
-<wire x1="66.04" y1="160.02" x2="66.04" y2="180.34" width="0.1524" layer="91"/>
+<wire x1="66.04" y1="160.02" x2="66.04" y2="182.88" width="0.1524" layer="91"/>
 <wire x1="33.02" y1="182.88" x2="66.04" y2="182.88" width="0.1524" layer="91"/>
-<wire x1="66.04" y1="182.88" x2="66.04" y2="180.34" width="0.1524" layer="91"/>
 <junction x="33.02" y="182.88"/>
+<pinref part="REG_BRIGHT" gate="G$1" pin="2"/>
+<wire x1="35.56" y1="177.8" x2="33.02" y2="177.8" width="0.1524" layer="91"/>
+<junction x="33.02" y="177.8"/>
 </segment>
 <segment>
@@
 </segment>
 </net>
-<net name="GND" class="0">
+<net name="GND" class="1">
 <segment>
 <pinref part="X1" gate="G$1" pin="VSS"/>
@@
 </segment>
 </net>
-<net name="N$14" class="0">
-<segment>
-<junction x="35.56" y="182.88"/>
-<pinref part="REG_BRIGHT" gate="G$1" pin="2"/>
-<wire x1="35.56" y1="177.8" x2="35.56" y2="182.88" width="0.1524" layer="91"/>
-</segment>
-</net>

Commit message: placa patrick atualizada
Parts:
- DOWN, RESET, UP: device switch-omron:10-XX -> switch-omron:40-XX
- R7: device bourns:3362P -> pot:3RP/1610N
Connections:
- net N$15: now also R7.A; no longer R7.1
- net N$16: now also R7.S; no longer R7.2
Changed lines of the file:
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@@
 <parts>
 <part name="FRAME1" library="frames" library_urn="urn:adsk.eagle:library:229" deviceset="A4P-LOC" device=""/>
-<part name="ARDUINO_NANO1" library="ArduinoNanoV30" deviceset="ARDUINO_NANO" device=""/>
-<part name="X1" library="adafruit" library_urn="urn:adsk.eagle:library:420" deviceset="HD44780LCD" device="-1602" package3d_urn="urn:adsk.eagle:package:6240760/1"/>
-<part name="REG_BRIGHT" library="adafruit" library_urn="urn:adsk.eagle:library:420" deviceset="FLIPFLOP-RES" device="" package3d_urn="urn:adsk.eagle:package:6240726/1"/>
-<part name="R2" library="adafruit" library_urn="urn:adsk.eagle:library:420" deviceset="FLIPFLOP-RES" device="" package3d_urn="urn:adsk.eagle:package:6240726/1"/>
-<part name="R3" library="adafruit" library_urn="urn:adsk.eagle:library:420" deviceset="FLIPFLOP-RES" device="" package3d_urn="urn:adsk.eagle:package:6240726/1"/>
-<part name="R4" library="adafruit" library_urn="urn:adsk.eagle:library:420" deviceset="FLIPFLOP-RES" device="" package3d_urn="urn:adsk.eagle:package:6240726/1"/>
-<part name="RESET" library="switch-omron" library_urn="urn:adsk.eagle:library:377" deviceset="10-XX" device="" package3d_urn="urn:adsk.eagle:package:27496/1"/>
-<part name="UP" library="switch-omron" library_urn="urn:adsk.eagle:library:377" deviceset="10-XX" device="" package3d_urn="urn:adsk.eagle:package:27496/1"/>
-<part name="SG1" library="buzzer" library_urn="urn:adsk.eagle:library:113" deviceset="F/CM12P" device="" package3d_urn="urn:adsk.eagle:package:5265/1"/>
-<part name="DOWN" library="switch-omron" library_urn="urn:adsk.eagle:library:377" deviceset="10-XX" device="" package3d_urn="urn:adsk.eagle:package:27496/1"/>
-<part name="R7" library="bourns" deviceset="3362" device="P"/>
+<part name="ARDUINO_NANO1" library="ArduinoNanoV30" deviceset="ARDUINO_NANO" device="" override_package3d_urn="urn:adsk.eagle:package:22034686/2" override_package_urn="urn:adsk.eagle:footprint:22034687/1"/>
+<part name="X1" library="adafruit" library_urn="urn:adsk.eagle:library:420" deviceset="HD44780LCD" device="-1602" package3d_urn="urn:adsk.eagle:package:6240760/1" override_package3d_urn="urn:adsk.eagle:package:22034966/2" override_package_urn="urn:adsk.eagle:footprint:6240114/1"/>
+<part name="REG_BRIGHT" library="adafruit" library_urn="urn:adsk.eagle:library:420" deviceset="FLIPFLOP-RES" device="" package3d_urn="urn:adsk.eagle:package:6240726/1" override_package3d_urn="urn:adsk.eagle:package:22222001/2" override_package_urn="urn:adsk.eagle:footprint:6240080/1"/>
+<part name="R2" library="adafruit" library_urn="urn:adsk.eagle:library:420" deviceset="FLIPFLOP-RES" device="" package3d_urn="urn:adsk.eagle:package:6240726/1" override_package3d_urn="urn:adsk.eagle:package:22222007/2" override_package_urn="urn:adsk.eagle:footprint:6240080/1"/>
+<part name="R3" library="adafruit" library_urn="urn:adsk.eagle:library:420" deviceset="FLIPFLOP-RES" device="" package3d_urn="urn:adsk.eagle:package:6240726/1" override_package3d_urn="urn:adsk.eagle:package:22034996/2" override_package_urn="urn:adsk.eagle:footprint:6240080/1"/>
+<part name="R4" library="adafruit" library_urn="urn:adsk.eagle:library:420" deviceset="FLIPFLOP-RES" device="" package3d_urn="urn:adsk.eagle:package:6240726/1" override_package3d_urn="urn:adsk.eagle:package:22221965/2" override_package_urn="urn:adsk.eagle:footprint:6240080/1"/>
+<part name="RESET" library="switch-omron" library_urn="urn:adsk.eagle:library:377" deviceset="40-XX" device="" package3d_urn="urn:adsk.eagle:package:27483/1" override_package3d_urn="urn:adsk.eagle:package:22221547/2" override_package_urn="urn:adsk.eagle:footprint:27470/1"/>
+<part name="UP" library="switch-omron" library_urn="urn:adsk.eagle:library:377" deviceset="40-XX" device="" package3d_urn="urn:adsk.eagle:package:27483/1" override_package3d_urn="urn:adsk.eagle:package:22035013/4" override_package_urn="urn:adsk.eagle:footprint:22221528/1"/>
+<part name="SG1" library="buzzer" library_urn="urn:adsk.eagle:library:113" deviceset="F/CM12P" device="" package3d_urn="urn:adsk.eagle:package:5265/1" override_package3d_urn="urn:adsk.eagle:package:22034983/2" override_package_urn="urn:adsk.eagle:footprint:5223/1"/>
+<part name="DOWN" library="switch-omron" library_urn="urn:adsk.eagle:library:377" deviceset="40-XX" device="" package3d_urn="urn:adsk.eagle:package:27483/1" override_package3d_urn="urn:adsk.eagle:package:22221545/2" override_package_urn="urn:adsk.eagle:footprint:27470/1"/>
+<part name="R7" library="pot" library_urn="urn:adsk.eagle:library:331" deviceset="3RP/1610N" device="" package3d_urn="urn:adsk.eagle:package:22726/1" override_package3d_urn="urn:adsk.eagle:package:22221551/2" override_package_urn="urn:adsk.eagle:footprint:22673/1"/>
 <part name="GND1" library="supply1" library_urn="urn:adsk.eagle:library:371" deviceset="GND" device=""/>
 <part name="GND2" library="supply1" library_urn="urn:adsk.eagle:library:371" deviceset="GND" device=""/>
@@
 <wire x1="116.84" y1="180.34" x2="86.36" y2="180.34" width="0.1524" layer="91"/>
 <wire x1="86.36" y1="180.34" x2="86.36" y2="185.42" width="0.1524" layer="91"/>
-<pinref part="R7" gate="G$1" pin="1"/>
+<pinref part="R7" gate="G$1" pin="A"/>
 </segment>
 </net>
 <net name="N$16" class="0">
 <segment>
-<pinref part="R7" gate="G$1" pin="2"/>
+<pinref part="R7" gate="G$1" pin="S"/>
 <pinref part="SG1" gate="G$1" pin="1"/>
 <wire x1="91.44" y1="190.5" x2="91.44" y2="200.66" width="0.1524" layer="91"/>
@@
 packages will not be understood (or retained) with this version.
 </note>
+<note version="9.4" severity="warning">
+Since Version 9.4, EAGLE supports the overriding of 3D packages
+in schematics and board files. Those overridden 3d packages
+will not be understood (or retained) with this version.
+</note>
 </compatibility>
