File: Esquematicos/Eagle/Phineas.sch (EAGLE design)
At the start: 11 parts

Commit message: Alterando Esquemático Phineas
Parts:
- renumbered S1 to PULAR, S2 to DESCER, S3 to RESET, SG1 to BUZZER
Connections:
- net N$10 renamed VCC
- net N$17 renamed GND

Commit message: Ajeitando esquemático Phineas
Parts:
- BUZZER: value F/EE21P -> F/QMB; device buzzer:F/EE21P -> buzzer:F/QMB
- DESCER, PULAR, RESET: device switch-omron:10-XX -> switch-omron:40-XX
- R1, R2, R3, R4: device rcl:R-US_0204/7 -> rcl:R-US_0207/10
- R5: device pot:TRIM_US-CIP20C-6MM -> pot:3RP/1610N
Connections:
- removed net N$16: BUZZER.2, R5.E
- new net N$10: BUZZER.-, R5.E
- new net N$15: R4.2, RESET.P1
- net GND: now also BUZZER.+; no longer BUZZER.1, R1.1
- net N$2: now also DIS1.CONTR; no longer PULAR.P1
- net N$3: now also PULAR.P1; no longer DESCER.P1
- net N$4: now also DESCER.P1; no longer RESET.P1
Other:
- moved on the sheet: R1, R2, R3, R4

Commit message: Alterando esquemático e board Phineas
Parts:
- PULAR: SPICEPREFIX (none) -> E
Changed lines of the file:
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@@
 </variantdefs>
 <classes>
-<class number="0" name="default" width="0" drill="0">
+<class number="0" name="default" width="0.508" drill="0">
+</class>
+<class number="1" name="alimentacao" width="1.016" drill="0">
 </class>
 </classes>
 <parts>
 <part name="FRAME1" library="frames" library_urn="urn:adsk.eagle:library:229" deviceset="A4P-LOC" device=""/>
-<part name="ARDUINO_NANO1" library="ArduinoNanoV30" deviceset="ARDUINO_NANO" device=""/>
-<part name="DIS1" library="display-lcd" library_urn="urn:adsk.eagle:library:214" deviceset="TUXGR_16X2_R2" device="" package3d_urn="urn:adsk.eagle:package:13139/1"/>
+<part name="ARDUINO_NANO1" library="ArduinoNanoV30" deviceset="ARDUINO_NANO" device="" override_package3d_urn="urn:adsk.eagle:package:22547936/2" override_package_urn="urn:adsk.eagle:footprint:22547943/1"/>
+<part name="DIS1" library="display-lcd" library_urn="urn:adsk.eagle:library:214" deviceset="TUXGR_16X2_R2" device="" package3d_urn="urn:adsk.eagle:package:13139/1" override_package3d_urn="urn:adsk.eagle:package:22547731/2" override_package_urn="urn:adsk.eagle:footprint:13120/1"/>
 <part name="GND2" library="supply1" library_urn="urn:adsk.eagle:library:371" deviceset="GND" device=""/>
 <part name="GND3" library="supply1" library_urn="urn:adsk.eagle:library:371" deviceset="GND" device=""/>
@@
 <part name="GND1" library="supply1" library_urn="urn:adsk.eagle:library:371" deviceset="GND" device=""/>
 <part name="GND6" library="supply1" library_urn="urn:adsk.eagle:library:371" deviceset="GND" device=""/>
-<part name="BUZZER" library="buzzer" library_urn="urn:adsk.eagle:library:113" deviceset="F/QMB" device="" package3d_urn="urn:adsk.eagle:package:5270/1"/>
-<part name="R5" library="pot" library_urn="urn:adsk.eagle:library:331" deviceset="3RP/1610N" device="" package3d_urn="urn:adsk.eagle:package:22726/1"/>
-<part name="R1" library="rcl" library_urn="urn:adsk.eagle:library:334" deviceset="R-US_" device="0207/10" package3d_urn="urn:adsk.eagle:package:23491/2"/>
-<part name="R2" library="rcl" library_urn="urn:adsk.eagle:library:334" deviceset="R-US_" device="0207/10" package3d_urn="urn:adsk.eagle:package:23491/2"/>
-<part name="R3" library="rcl" library_urn="urn:adsk.eagle:library:334" deviceset="R-US_" device="0207/10" package3d_urn="urn:adsk.eagle:package:23491/2"/>
-<part name="R4" library="rcl" library_urn="urn:adsk.eagle:library:334" deviceset="R-US_" device="0207/10" package3d_urn="urn:adsk.eagle:package:23491/2"/>
-<part name="PULAR" library="switch-omron" library_urn="urn:adsk.eagle:library:377" deviceset="40-XX" device="" package3d_urn="urn:adsk.eagle:package:27483/1"/>
-<part name="DESCER" library="switch-omron" library_urn="urn:adsk.eagle:library:377" deviceset="40-XX" device="" package3d_urn="urn:adsk.eagle:package:27483/1"/>
-<part name="RESET" library="switch-omron" library_urn="urn:adsk.eagle:library:377" deviceset="40-XX" device="" package3d_urn="urn:adsk.eagle:package:27483/1"/>
+<part name="BUZZER" library="buzzer" library_urn="urn:adsk.eagle:library:113" deviceset="F/QMB" device="" package3d_urn="urn:adsk.eagle:package:5270/1" override_package3d_urn="urn:adsk.eagle:package:22548628/3" override_package_urn="urn:adsk.eagle:footprint:5226/1"/>
+<part name="R5" library="pot" library_urn="urn:adsk.eagle:library:331" deviceset="3RP/1610N" device="" package3d_urn="urn:adsk.eagle:package:22726/1" override_package3d_urn="urn:adsk.eagle:package:22548630/2" override_package_urn="urn:adsk.eagle:footprint:22673/1"/>
+<part name="R1" library="rcl" library_urn="urn:adsk.eagle:library:334" deviceset="R-US_" device="0207/10" package3d_urn="urn:adsk.eagle:package:23491/2" override_package3d_urn="urn:adsk.eagle:package:22547733/2" override_package_urn="urn:adsk.eagle:footprint:22992/1"/>
+<part name="R2" library="rcl" library_urn="urn:adsk.eagle:library:334" deviceset="R-US_" device="0207/10" package3d_urn="urn:adsk.eagle:package:23491/2" override_package3d_urn="urn:adsk.eagle:package:22548606/2" override_package_urn="urn:adsk.eagle:footprint:22992/1"/>
+<part name="R3" library="rcl" library_urn="urn:adsk.eagle:library:334" deviceset="R-US_" device="0207/10" package3d_urn="urn:adsk.eagle:package:23491/2" override_package3d_urn="urn:adsk.eagle:package:22548620/2" override_package_urn="urn:adsk.eagle:footprint:22992/1"/>
+<part name="R4" library="rcl" library_urn="urn:adsk.eagle:library:334" deviceset="R-US_" device="0207/10" package3d_urn="urn:adsk.eagle:package:23491/2" override_package3d_urn="urn:adsk.eagle:package:22548624/2" override_package_urn="urn:adsk.eagle:footprint:22992/1"/>
+<part name="PULAR" library="switch-omron" library_urn="urn:adsk.eagle:library:377" deviceset="40-XX" device="" package3d_urn="urn:adsk.eagle:package:27483/1" override_package3d_urn="urn:adsk.eagle:package:22548614/3" override_package_urn="urn:adsk.eagle:footprint:27470/1">
+<attribute name="SPICEPREFIX" value="E"/>
+</part>
+<part name="DESCER" library="switch-omron" library_urn="urn:adsk.eagle:library:377" deviceset="40-XX" device="" package3d_urn="urn:adsk.eagle:package:27483/1" override_package3d_urn="urn:adsk.eagle:package:22548618/2" override_package_urn="urn:adsk.eagle:footprint:27470/1"/>
+<part name="RESET" library="switch-omron" library_urn="urn:adsk.eagle:library:377" deviceset="40-XX" device="" package3d_urn="urn:adsk.eagle:package:27483/1" override_package3d_urn="urn:adsk.eagle:package:22548622/2" override_package_urn="urn:adsk.eagle:footprint:27470/1"/>
 </parts>
 <sheets>
@@
 </segment>
 </net>
-<net name="GND" class="0">
+<net name="GND" class="1">
 <segment>
 <pinref part="ARDUINO_NANO1" gate="G$1" pin="GND@1"/>
@@
 </segment>
 </net>
-<net name="VCC" class="0">
+<net name="VCC" class="1">
 <segment>
 <wire x1="121.92" y1="220.98" x2="121.92" y2="215.9" width="0.1524" layer="91"/>
@@
 packages will not be understood (or retained) with this version.
 </note>
+<note version="9.4" severity="warning">
+Since Version 9.4, EAGLE supports the overriding of 3D packages
+in schematics and board files. Those overridden 3d packages
+will not be understood (or retained) with this version.
+</note>
 <note version="8.4" severity="warning">
